Commit message: added tf link for raspicam

File: urdf/common_properties.urdf.xacro (robot description, xacro)
@@ -11,4 +11,5 @@
   <xacro:property name="first_tier_to_second_tier" value="0.105"/>
   <xacro:property name="second_tier_to_third_tier" value="0.092"/>
+  <xacro:property name="second_tier_to_rpicam" value="0.115"/>
   <xacro:property name="third_tier_to_slam_tier" value="0.192"/>
 </robot>

File: urdf/tango.urdf.xacro (robot description, xacro)
@@ -28,4 +28,5 @@
   <xacro:create_fixed_link_joint prefix="second_tier" parent="first_tier_link" joint_xyz="0 0 ${first_tier_to_second_tier}" joint_rpy="0 0 0"/>
   <xacro:create_fixed_link_joint prefix="third_tier" parent="second_tier_link" joint_xyz="0 0 ${second_tier_to_third_tier}" joint_rpy="0 0 0"/>
+  <xacro:create_fixed_link_joint prefix="rpicamera" parent="second_tier_link" joint_xyz="${second_tier_to_rpicam} 0 0" joint_rpy="0 0 0"/>
   <xacro:create_fixed_link_joint prefix="slam_tier" parent="third_tier_link" joint_xyz="-0.115 0 ${third_tier_to_slam_tier}" joint_rpy="0 0 0"/>
   <xacro:if value="$(arg arc)">

Commit message: added zed camera base link

File: urdf/common_properties.urdf.xacro (robot description, xacro)
@@ -11,5 +11,6 @@
   <xacro:property name="first_tier_to_second_tier" value="0.105"/>
   <xacro:property name="second_tier_to_third_tier" value="0.092"/>
-  <xacro:property name="second_tier_to_rpicam" value="0.115"/>
+  <xacro:property name="first_tier_to_zed" value="0.155"/>
+  <xacro:property name="first_tier_to_zed_height" value="0.025"/>
   <xacro:property name="third_tier_to_slam_tier" value="0.192"/>
 </robot>

File: urdf/tango.urdf.xacro (robot description, xacro)
@@ -28,5 +28,5 @@
   <xacro:create_fixed_link_joint prefix="second_tier" parent="first_tier_link" joint_xyz="0 0 ${first_tier_to_second_tier}" joint_rpy="0 0 0"/>
   <xacro:create_fixed_link_joint prefix="third_tier" parent="second_tier_link" joint_xyz="0 0 ${second_tier_to_third_tier}" joint_rpy="0 0 0"/>
-  <xacro:create_fixed_link_joint prefix="rpicamera" parent="second_tier_link" joint_xyz="${second_tier_to_rpicam} 0 0" joint_rpy="0 0 0"/>
+  <xacro:create_fixed_link_joint prefix="zedcamera" parent="first_tier_link" joint_xyz="${first_tier_to_zed} 0 ${first_tier_to_zed_height}" joint_rpy="0 0.226893 0"/>
   <xacro:create_fixed_link_joint prefix="slam_tier" parent="third_tier_link" joint_xyz="-0.115 0 ${third_tier_to_slam_tier}" joint_rpy="0 0 0"/>
   <xacro:if value="$(arg arc)">
